Commit message: working URDF and rviz display

File: ros2_ws/src/pantographe_description/urdf/pantographe_generated.urdf (robot description, URDF)
Before this commit: robot pantographe, 9 links, 8 joints
Links:
- removed link link1_pivot
- removed link link2_pivot
- removed link link3_pivot
- removed link link4_pivot
- link base: geometry collision mesh filename=package://pantographe_description/meshes/bati.dae; visual mesh filename=package://pantographe_description/meshes/bati.dae
Joints:
- removed joint link1_fixed
- removed joint link2_fixed
- removed joint link3_fixed
- removed joint link4_fixed
- joint joint1: child link1_pivot -> link1
- joint joint2: child link2_pivot -> link2
- joint joint3: child link3_pivot -> link3
- joint joint4: child link4_pivot -> link4
